Commit message: Modify urdf to add oak-d camera

File: scout_description/urdf/scout_v2.urdf (robot description, URDF)
Before this commit: robot scout_v2, 7 links, 6 joints
Links:
- added link oak-d_frame
- added link oak_model_origin; visual mesh filename=package://depthai_bridge/urdf/models/OAK-D-PRO.stl
- link front_left_wheel_link: geometry collision cylinder length=0.11653 radius=0.16459; visual mesh filename=package://scout_description/meshes/scout_v2/wheel_type2.dae
- link front_right_wheel_link: geometry collision cylinder length=0.11653 radius=0.16459; visual mesh filename=package://scout_description/meshes/scout_v2/wheel_type1.dae
- link rear_left_wheel_link: geometry collision cylinder length=0.11653 radius=0.16459; visual mesh filename=package://scout_description/meshes/scout_v2/wheel_type1.dae
- link rear_right_wheel_link: geometry collision cylinder length=0.11653 radius=0.16459; visual mesh filename=package://scout_description/meshes/scout_v2/wheel_type2.dae
Joints:
- added joint oak_center_joint: type fixed, parent base_link, child oak-d_frame, origin xyz=0.4 0.0 0.25 rpy=0 0 0
- added joint oak_model_origin_joint: type fixed, parent oak-d_frame, child oak_model_origin, origin xyz=0 0 0 rpy=1.5708 0 1.5708

File: scout_description/urdf/scout_v2.xacro (robot description, xacro)
@@ -7,4 +7,5 @@
     <!-- Variables -->
     <xacro:property name="M_PI" value="3.14159"/>
+    <xacro:property name="baseline" value="0.075" />
     <!-- Vehicle Geometries -->
     <xacro:property name="base_x_size" value="0.9250000" />
@@ -70,3 +71,74 @@
         <origin xyz="${-wheelbase/2} ${-track/2} ${wheel_vertical_offset}" rpy="3.14 0 0" />
     </xacro:scout_wheel_type2>
+    <!-- base_link of the sensor-->
+    <link name="oak-d_frame"/>
+    <joint name="oak_center_joint" type="fixed">
+        <parent link="base_link"/>
+        <child link="oak-d_frame"/>
+        <origin xyz="0.4 0.0 0.25" rpy="0 0 0" />
+    </joint>
+<!-- device Center -->
+    <link name="oak_model_origin">
+        <visual>
+            <origin xyz="0 0 0" rpy="0 0 0"/>
+            <geometry>
+                <mesh filename="package://depthai_bridge/urdf/models/OAK-D-PRO.stl" />
+                <material name="mat">
+                <color rgba="0.8 0.8 0.8 0.8"/>
+                <!-- TODO: FIX COLORING -->
+            </material>
+            </geometry>
+        </visual>
+    </link>
+    <joint name="oak_model_origin_joint" type="fixed">
+        <parent link="oak-d_frame"/>
+        <child link="oak_model_origin"/>
+        <origin xyz="0 0 0" rpy="1.5708 0 1.5708" />
+    </joint>
+    <!-- IMU -->
+        <link name="oak_imu_frame" />
+        <joint name="oak_imu_joint" type="fixed">
+            <parent link="oak-d_frame"/>
+            <child link="oak_imu_frame"/>
+            <origin xyz="0 0 0" rpy="0 0 0" />
+        </joint>
+<!-- RGB Camera -->
+    <link name="oak_rgb_camera_frame" />
+    <joint name="oak_rgb_camera_joint" type="fixed">
+        <parent link="oak-d_frame"/>
+        <child link="oak_rgb_camera_frame"/>
+        <origin xyz="0 0 0" rpy="0 0 0" />
+    </joint>
+    <link name="oak_rgb_camera_optical_frame"/>
+    <joint name="oak_rgb_camera_optical_joint" type="fixed">
+        <origin xyz="0 0 0" rpy="-${M_PI/2} 0.0 -${M_PI/2}"/>
+        <parent link="oak_rgb_camera_frame"/>
+        <child link="oak_rgb_camera_optical_frame"/>
+    </joint>
+<!-- Left Camera -->
+    <link name="oak_left_camera_frame" />
+    <joint name="oak_left_camera_joint" type="fixed">
+        <parent link="oak-d_frame"/>
+        <child link="oak_left_camera_frame"/>
+        <origin xyz="0 ${baseline/2} 0" rpy="0 0 0" />
+    </joint>
+    <link name="oak_left_camera_optical_frame"/>
+    <joint name="oak_left_camera_optical_joint" type="fixed">
+        <origin xyz="0 0 0" rpy="-${M_PI/2} 0.0 -${M_PI/2}"/>
+        <parent link="oak_left_camera_frame"/>
+        <child link="oak_left_camera_optical_frame"/>
+    </joint>
+<!-- right Camera -->
+    <link name="oak_right_camera_frame" />
+    <joint name="oak_right_camera_joint" type="fixed">
+        <parent link="oak-d_frame"/>
+        <child link="oak_right_camera_frame"/>
+        <origin xyz="0 -${baseline/2} 0" rpy="0 0 0" />
+    </joint>
+    <link name="oak_right_camera_optical_frame"/>
+    <joint name="oak_right_camera_optical_joint" type="fixed">
+        <origin xyz="0 0 0" rpy="-${M_PI/2} 0.0 -${M_PI/2}"/>
+        <parent link="oak_right_camera_frame"/>
+        <child link="oak_right_camera_optical_frame"/>
+    </joint>
 </robot>

Commit message: Avoid writing TODOs tags in comments

File: scout_description/urdf/scout_v2.urdf (robot description, URDF)
Before this commit: robot scout_v2, 9 links, 8 joints
Links:
- added link oak_imu_frame
- added link oak_left_camera_frame
- added link oak_left_camera_optical_frame
- added link oak_rgb_camera_frame
- added link oak_rgb_camera_optical_frame
- added link oak_right_camera_frame
- added link oak_right_camera_optical_frame
Joints:
- added joint oak_imu_joint: type fixed, parent oak-d_frame, child oak_imu_frame, origin xyz=0 0 0 rpy=0 0 0
- added joint oak_left_camera_joint: type fixed, parent oak-d_frame, child oak_left_camera_frame, origin xyz=0 0.0375 0 rpy=0 0 0
- added joint oak_left_camera_optical_joint: type fixed, parent oak_left_camera_frame, child oak_left_camera_optical_frame, origin xyz=0 0 0 rpy=-1.570795 0.0 -1.570795
- added joint oak_rgb_camera_joint: type fixed, parent oak-d_frame, child oak_rgb_camera_frame, origin xyz=0 0 0 rpy=0 0 0
- added joint oak_rgb_camera_optical_joint: type fixed, parent oak_rgb_camera_frame, child oak_rgb_camera_optical_frame, origin xyz=0 0 0 rpy=-1.570795 0.0 -1.570795
- added joint oak_right_camera_joint: type fixed, parent oak-d_frame, child oak_right_camera_frame, origin xyz=0 -0.0375 0 rpy=0 0 0
- added joint oak_right_camera_optical_joint: type fixed, parent oak_right_camera_frame, child oak_right_camera_optical_frame, origin xyz=0 0 0 rpy=-1.570795 0.0 -1.570795

File: scout_description/urdf/scout_v2.xacro (robot description, xacro)
@@ -84,9 +84,8 @@
             <geometry>
                 <mesh filename="package://depthai_bridge/urdf/models/OAK-D-PRO.stl" />
-                <material name="mat">
+            </geometry>
+            <material name="mat">
                 <color rgba="0.8 0.8 0.8 0.8"/>
-                <!-- TODO: FIX COLORING -->
             </material>
-            </geometry>
         </visual>
     </link>
