Commit message: URDF修正

File: scout_description/urdf/scout_mini.urdf (robot description, URDF)
Before this commit: robot scout_mini, 8 links, 7 joints
Joints:
- joint front_left_wheel: type continuous -> fixed
- joint front_right_wheel: type continuous -> fixed
- joint rear_left_wheel: type continuous -> fixed
- joint rear_right_wheel: type continuous -> fixed

File: scout_description/urdf/scout_mini_wheel.xacro (robot description, xacro)
@@ -24,5 +24,5 @@
             </collision>
         </link>
-        <joint name="${wheel_prefix}_wheel" type="continuous">
+        <joint name="${wheel_prefix}_wheel" type="fixed">
             <parent link="base_link"/>
             <child link="${wheel_prefix}_wheel_link"/>
